Commit message: add logo

File: urdf/MAGICBOT.urdf (robot description, URDF)
Before this commit: robot Magicbot-Gen1, 35 links, 34 joints
Links:
- added link logo_link; visual mesh filename=package://magicbot_gen1_description/meshes/logo_link.STL scale=1.5 1.5 1.5
Joints:
- added joint logo_joint: type fixed, parent link_wy, child logo_link, origin xyz=-0.042 0 -0.272 rpy=0 0 0

File: urdf/MAGICBOT_with_hand.urdf (robot description, URDF)
Before this commit: robot Magicbot-Gen1, 57 links, 56 joints
Links:
- added link logo_link; visual mesh filename=package://magicbot_gen1_description/meshes/logo_link.STL scale=1.5 1.5 1.5
Joints:
- added joint logo_joint: type fixed, parent link_wy, child logo_link, origin xyz=-0.042 0 -0.272 rpy=0 0 0

Commit message: remove moveit config

File: urdf/MAGICBOT.urdf (robot description, URDF)
Before this commit: robot Magicbot-Gen1, 36 links, 35 joints
Links:
- link LINK_ANKLE_PITCH_L: geometry collision mesh filename=package://magicbot-gen1_description/meshes/LINK_ANKLE_PITCH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; visual mesh filename=package://magicbot-gen1_description/meshes/LINK_ANKLE_PITCH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
- link LINK_ANKLE_PITCH_R: geometry collision mesh filename=package://magicbot-gen1_description/meshes/LINK_ANKLE_PITCH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; visual mesh filename=package://magicbot-gen1_description/meshes/LINK_ANKLE_PITCH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
- link LINK_ANKLE_ROLL_L: geometry collision mesh filename=package://magicbot-gen1_description/meshes/LINK_ANKLE_ROLL_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; visual mesh filename=package://magicbot-gen1_description/meshes/LINK_ANKLE_ROLL_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
- link LINK_ANKLE_ROLL_R: geometry collision mesh filename=package://magicbot-gen1_description/meshes/LINK_ANKLE_ROLL_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; visual mesh filename=package://magicbot-gen1_description/meshes/LINK_ANKLE_ROLL_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
- link LINK_HIP_PITCH_L: geometry collision mesh filename=package://magicbot-gen1_description/meshes/LINK_HIP_PITCH_L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; visual mesh filename=package://magicbot-gen1_description/meshes/LINK_HIP_PITCH_L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
- link LINK_HIP_PITCH_R: geometry collision mesh filename=package://magicbot-gen1_description/meshes/LINK_HIP_PITCH_R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; visual mesh filename=package://magicbot-gen1_description/meshes/LINK_HIP_PITCH_R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
- link LINK_HIP_ROLL_L: geometry collision mesh filename=package://magicbot-gen1_description/meshes/LINK_HIP_ROLL_L.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; visual mesh filename=package://magicbot-gen1_description/meshes/LINK_HIP_ROLL_L.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
- link LINK_HIP_ROLL_R: geometry collision mesh filename=package://magicbot-gen1_description/meshes/LINK_HIP_ROLL_R.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; visual mesh filename=package://magicbot-gen1_description/meshes/LINK_HIP_ROLL_R.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
- link LINK_HIP_YAW_L: geometry collision mesh filename=package://magicbot-gen1_description/meshes/LINK_HIP_YAW_L.S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; visual mesh filename=package://magicbot-gen1_description/meshes/LINK_HIP_YAW_L.S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
- link LINK_HIP_YAW_R: geometry collision mesh filename=package://magicbot-gen1_description/meshes/LINK_HIP_YAW_R.S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; visual mesh filename=package://magicbot-gen1_description/meshes/LINK_HIP_YAW_R.S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
- link LINK_KNEE_PITCH_L: geometry collision mesh filename=package://magicbot-gen1_description/meshes/LINK_KNEE_PITCH_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; visual mesh filename=package://magicbot-gen1_description/meshes/LINK_KNEE_PITCH_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
- link LINK_KNEE_PITCH_R: geometry collision mesh filename=package://magicbot-gen1_description/meshes/LINK_KNEE_PITCH_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; visual mesh filename=package://magicbot-gen1_description/meshes/LINK_KNEE_PITCH_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
- link link_hp: geometry collision mesh filename=package://magicbot-gen1_description/meshes/link_hp.STL; visual mesh filename=package://magicbot-gen1_description/meshes/link_hp.STL
- link link_hy: geometry collision mesh filename=package://magicbot-gen1_description/meshes/link_hy.STL; visual mesh filename=package://magicbot-gen1_description/meshes/link_hy.STL
- link link_la1: geometry collision mesh filename=package://magicbot-gen1_description/meshes/link_la1.STL; visual mesh filename=package://magicbot-gen1_description/meshes/link_la1.STL
- link link_la2: geometry collision mesh filename=package://magicbot-gen1_description/meshes/link_la2.STL; visual mesh filename=package://magicbot-gen1_description/meshes/link_la2.STL
- link link_la3: geometry collision mesh filename=package://magicbot-gen1_description/meshes/link_la3.STL; visual mesh filename=package://magicbot-gen1_description/meshes/link_la3.STL
- link link_la4: geometry collision mesh filename=package://magicbot-gen1_description/meshes/link_la4.STL; visual mesh filename=package://magicbot-gen1_description/meshes/link_la4.STL
- link link_la5: geometry collision mesh filename=package://magicbot-gen1_description/meshes/link_la5.STL; visual mesh filename=package://magicbot-gen1_description/meshes/link_la5.STL
- link link_la6: geometry collision mesh filename=package://magicbot-gen1_description/meshes/link_la6.STL; visual mesh filename=package://magicbot-gen1_description/meshes/link_la6.STL
- link link_la7: geometry collision mesh filename=package://magicbot-gen1_description/meshes/link_la7.STL; visual mesh filename=package://magicbot-gen1_description/meshes/link_la7.STL
- link link_ra1: geometry collision mesh filename=package://magicbot-gen1_description/meshes/link_ra1.STL; visual mesh filename=package://magicbot-gen1_description/meshes/link_ra1.STL
- link link_ra2: geometry collision mesh filename=package://magicbot-gen1_description/meshes/link_ra2.STL; visual mesh filename=package://magicbot-gen1_description/meshes/link_ra2.STL
- link link_ra3: geometry collision mesh filename=package://magicbot-gen1_description/meshes/link_ra3.STL; visual mesh filename=package://magicbot-gen1_description/meshes/link_ra3.STL
- link link_ra4: geometry collision mesh filename=package://magicbot-gen1_description/meshes/link_ra4.STL; visual mesh filename=package://magicbot-gen1_description/meshes/link_ra4.STL
- link link_ra5: geometry collision mesh filename=package://magicbot-gen1_description/meshes/link_ra5.STL; visual mesh filename=package://magicbot-gen1_description/meshes/link_ra5.STL
- link link_ra6: geometry collision mesh filename=package://magicbot-gen1_description/meshes/link_ra6.STL; visual mesh filename=package://magicbot-gen1_description/meshes/link_ra6.STL
- link link_ra7: geometry collision mesh filename=package://magicbot-gen1_description/meshes/link_ra7.STL; visual mesh filename=package://magicbot-gen1_description/meshes/link_ra7.STL
- link link_wr: geometry collision mesh filename=package://magicbot-gen1_description/meshes/link_wr.STL; visual mesh filename=package://magicbot-gen1_description/meshes/link_wr.STL
- link link_wy: geometry collision mesh filename=package://magicbot-gen1_description/meshes/link_wy.STL; visual mesh filename=package://magicbot-gen1_description/meshes/link_wy.STL
- link logo_link: geometry visual mesh filename=package://magicbot-gen1_description/meshes/logo_link.STL scale=1.5 1.5 1.5
- link pelvis: geometry collision mesh filename=package://magicbot-gen1_description/meshes/pelvis.STL; visual mesh filename=package://magicbot-gen1_description/meshes/pelvis.STL

File: urdf/MAGICBOT_with_hand.urdf (robot description, URDF)
Before this commit: robot Magicbot-Gen1, 58 links, 57 joints
Links:
- link LINK_ANKLE_PITCH_L: geometry collision mesh filename=package://magicbot-gen1_description/meshes/LINK_ANKLE_PITCH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; visual mesh filename=package://magicbot-gen1_description/meshes/LINK_ANKLE_PITCH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
- link LINK_ANKLE_PITCH_R: geometry collision mesh filename=package://magicbot-gen1_description/meshes/LINK_ANKLE_PITCH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; visual mesh filename=package://magicbot-gen1_description/meshes/LINK_ANKLE_PITCH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
- link LINK_ANKLE_ROLL_L: geometry collision mesh filename=package://magicbot-gen1_description/meshes/LINK_ANKLE_ROLL_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; visual mesh filename=package://magicbot-gen1_description/meshes/LINK_ANKLE_ROLL_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
- link LINK_ANKLE_ROLL_R: geometry collision mesh filename=package://magicbot-gen1_description/meshes/LINK_ANKLE_ROLL_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; visual mesh filename=package://magicbot-gen1_description/meshes/LINK_ANKLE_ROLL_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
- link LINK_HIP_PITCH_L: geometry collision mesh filename=package://magicbot-gen1_description/meshes/LINK_HIP_PITCH_L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; visual mesh filename=package://magicbot-gen1_description/meshes/LINK_HIP_PITCH_L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
- link LINK_HIP_PITCH_R: geometry collision mesh filename=package://magicbot-gen1_description/meshes/LINK_HIP_PITCH_R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; visual mesh filename=package://magicbot-gen1_description/meshes/LINK_HIP_PITCH_R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
- link LINK_HIP_ROLL_L: geometry collision mesh filename=package://magicbot-gen1_description/meshes/LINK_HIP_ROLL_L.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; visual mesh filename=package://magicbot-gen1_description/meshes/LINK_HIP_ROLL_L.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
- link LINK_HIP_ROLL_R: geometry collision mesh filename=package://magicbot-gen1_description/meshes/LINK_HIP_ROLL_R.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; visual mesh filename=package://magicbot-gen1_description/meshes/LINK_HIP_ROLL_R.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
- link LINK_HIP_YAW_L: geometry collision mesh filename=package://magicbot-gen1_description/meshes/LINK_HIP_YAW_L.S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; visual mesh filename=package://magicbot-gen1_description/meshes/LINK_HIP_YAW_L.S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
- link LINK_HIP_YAW_R: geometry collision mesh filename=package://magicbot-gen1_description/meshes/LINK_HIP_YAW_R.S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; visual mesh filename=package://magicbot-gen1_description/meshes/LINK_HIP_YAW_R.S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
- link LINK_KNEE_PITCH_L: geometry collision mesh filename=package://magicbot-gen1_description/meshes/LINK_KNEE_PITCH_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; visual mesh filename=package://magicbot-gen1_description/meshes/LINK_KNEE_PITCH_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
- link LINK_KNEE_PITCH_R: geometry collision mesh filename=package://magicbot-gen1_description/meshes/LINK_KNEE_PITCH_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; visual mesh filename=package://magicbot-gen1_description/meshes/LINK_KNEE_PITCH_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
- link forefinger1_Link: geometry collision mesh filename=package://magicbot-gen1_description/meshes/forefinger1_Link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; visual mesh filename=package://magicbot-gen1_description/meshes/forefinger1_Link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
- link forefinger1_Link_R: geometry collision mesh filename=package://magicbot-gen1_description/meshes/forefinger1_Link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; visual mesh filename=package://magicbot-gen1_description/meshes/forefinger1_Link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
- link forefinger2_Link: geometry collision mesh filename=package://magicbot-gen1_description/meshes/forefinger2_Link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; visual mesh filename=package://magicbot-gen1_description/meshes/forefinger2_Link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
- link forefinger2_Link_R: geometry collision mesh filename=package://magicbot-gen1_description/meshes/forefinger2_Link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; visual mesh filename=package://magicbot-gen1_description/meshes/forefinger2_Link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
- link hand_Link_R: geometry collision mesh filename=package://magicbot-gen1_description/meshes/hand_Link_R.STL; visual mesh filename=package://magicbot-gen1_description/meshes/hand_Link_R.STL
- link hand_link: geometry collision mesh filename=package://magicbot-gen1_description/meshes/hand_link.STL; visual mesh filename=package://magicbot-gen1_description/meshes/hand_link.STL
- link link_hp: geometry collision mesh filename=package://magicbot-gen1_description/meshes/link_hp.STL; visual mesh filename=package://magicbot-gen1_description/meshes/link_hp.STL
- link link_hy: geometry collision mesh filename=package://magicbot-gen1_description/meshes/link_hy.STL; visual mesh filename=package://magicbot-gen1_description/meshes/link_hy.STL
- link link_la1: geometry collision mesh filename=package://magicbot-gen1_description/meshes/link_la1.STL; visual mesh filename=package://magicbot-gen1_description/meshes/link_la1.STL
- link link_la2: geometry collision mesh filename=package://magicbot-gen1_description/meshes/link_la2.STL; visual mesh filename=package://magicbot-gen1_description/meshes/link_la2.STL
- link link_la3: geometry collision mesh filename=package://magicbot-gen1_description/meshes/link_la3.STL; visual mesh filename=package://magicbot-gen1_description/meshes/link_la3.STL
- link link_la4: geometry collision mesh filename=package://magicbot-gen1_description/meshes/link_la4.STL; visual mesh filename=package://magicbot-gen1_description/meshes/link_la4.STL
- link link_la5: geometry collision mesh filename=package://magicbot-gen1_description/meshes/link_la5.STL; visual mesh filename=package://magicbot-gen1_description/meshes/link_la5.STL
- link link_la6: geometry collision mesh filename=package://magicbot-gen1_description/meshes/link_la6.STL; visual mesh filename=package://magicbot-gen1_description/meshes/link_la6.STL
- link link_ra1: geometry collision mesh filename=package://magicbot-gen1_description/meshes/link_ra1.STL; visual mesh filename=package://magicbot-gen1_description/meshes/link_ra1.STL
- link link_ra2: geometry collision mesh filename=package://magicbot-gen1_description/meshes/link_ra2.STL; visual mesh filename=package://magicbot-gen1_description/meshes/link_ra2.STL
- link link_ra3: geometry collision mesh filename=package://magicbot-gen1_description/meshes/link_ra3.STL; visual mesh filename=package://magicbot-gen1_description/meshes/link_ra3.STL
- link link_ra4: geometry collision mesh filename=package://magicbot-gen1_description/meshes/link_ra4.STL; visual mesh filename=package://magicbot-gen1_description/meshes/link_ra4.STL
- link link_ra5: geometry collision mesh filename=package://magicbot-gen1_description/meshes/link_ra5.STL; visual mesh filename=package://magicbot-gen1_description/meshes/link_ra5.STL
- link link_ra6: geometry collision mesh filename=package://magicbot-gen1_description/meshes/link_ra6.STL; visual mesh filename=package://magicbot-gen1_description/meshes/link_ra6.STL
- link link_wr: geometry collision mesh filename=package://magicbot-gen1_description/meshes/link_wr.STL; visual mesh filename=package://magicbot-gen1_description/meshes/link_wr.STL
- link link_wy: geometry collision mesh filename=package://magicbot-gen1_description/meshes/link_wy.STL; visual mesh filename=package://magicbot-gen1_description/meshes/link_wy.STL
- link little1_Link: geometry collision mesh filename=package://magicbot-gen1_description/meshes/little1_Link.STL; visual mesh filename=package://magicbot-gen1_description/meshes/little1_Link.STL
- link little1_Link_R: geometry collision mesh filename=package://magicbot-gen1_description/meshes/little1_Link_R.S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; visual mesh filename=package://magicbot-gen1_description/meshes/little1_Link_R.S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
- link little2_Link: geometry collision mesh filename=package://magicbot-gen1_description/meshes/little2_Link.STL; visual mesh filename=package://magicbot-gen1_description/meshes/little2_Link.STL
- link little2_Link_R: geometry collision mesh filename=package://magicbot-gen1_description/meshes/little2_Link_R.S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; visual mesh filename=package://magicbot-gen1_description/meshes/little2_Link_R.S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
- link logo_link: geometry visual mesh filename=package://magicbot-gen1_description/meshes/logo_link.STL scale=1.5 1.5 1.5
- link middle1_Link: geometry collision mesh filename=package://magicbot-gen1_description/meshes/middle1_Link.STL; visual mesh filename=package://magicbot-gen1_description/meshes/middle1_Link.STL
- link middle1_Link_R: geometry collision mesh filename=package://magicbot-gen1_description/meshes/middle1_Link_R.S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; visual mesh filename=package://magicbot-gen1_description/meshes/middle1_Link_R.S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
- link middle2_Link: geometry collision mesh filename=package://magicbot-gen1_description/meshes/middle2_Link.STL; visual mesh filename=package://magicbot-gen1_description/meshes/middle2_Link.STL
- link middle2_Link_R: geometry collision mesh filename=package://magicbot-gen1_description/meshes/middle2_Link_R.S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; visual mesh filename=package://magicbot-gen1_description/meshes/middle2_Link_R.S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
- link pelvis: geometry collision mesh filename=package://magicbot-gen1_description/meshes/pelvis.STL; visual mesh filename=package://magicbot-gen1_description/meshes/pelvis.STL
- link ring1_Link: geometry collision mesh filename=package://magicbot-gen1_description/meshes/ring1_Link.STL; visual mesh filename=package://magicbot-gen1_description/meshes/ring1_Link.STL
- link ring1_Link_R: geometry collision mesh filename=package://magicbot-gen1_description/meshes/ring1_Link_R.STL; visual mesh filename=package://magicbot-gen1_description/meshes/ring1_Link_R.STL
- link ring2_Link: geometry collision mesh filename=package://magicbot-gen1_description/meshes/ring2_Link.STL; visual mesh filename=package://magicbot-gen1_description/meshes/ring2_Link.STL
- link ring2_Link_R: geometry collision mesh filename=package://magicbot-gen1_description/meshes/ring2_Link_R.STL; visual mesh filename=package://magicbot-gen1_description/meshes/ring2_Link_R.STL
- link thumb1_Link: geometry collision mesh filename=package://magicbot-gen1_description/meshes/thumb1_Link.STL; visual mesh filename=package://magicbot-gen1_description/meshes/thumb1_Link.STL
- link thumb1_Link_R: geometry collision mesh filename=package://magicbot-gen1_description/meshes/thumb1_Link_R.STL; visual mesh filename=package://magicbot-gen1_description/meshes/thumb1_Link_R.STL
- link thumb2_Link: geometry collision mesh filename=package://magicbot-gen1_description/meshes/thumb2_Link.STL; visual mesh filename=package://magicbot-gen1_description/meshes/thumb2_Link.STL
- link thumb2_Link_R: geometry collision mesh filename=package://magicbot-gen1_description/meshes/thumb2_Link_R.STL; visual mesh filename=package://magicbot-gen1_description/meshes/thumb2_Link_R.STL
- link thumb3_Link: geometry collision mesh filename=package://magicbot-gen1_description/meshes/thumb3_Link.STL; visual mesh filename=package://magicbot-gen1_description/meshes/thumb3_Link.STL
- link thumb3_Link_R: geometry collision mesh filename=package://magicbot-gen1_description/meshes/thumb3_Link_R.STL; visual mesh filename=package://magicbot-gen1_description/meshes/thumb3_Link_R.STL
